File: NMOS_SWITCH.kicad_pcb (KiCad board)
At the start: 2 copper layers, 35 x 25 mm, 22 parts, among them J1 Conn_01x02, J2 Conn_01x02, J3 Conn_01x02, Q1 Q_NPN_BCE, Q2 CSD18540Q5B, U1 BTS443P, U2 LM5050-1

Commit message: Adoption changes for engineering
Parts:
- added H2: MountingHole, MountingHole:MountingHole_3.2mm_M3, F.Cu at (142.4, 86.2)
- J2: footprint Connector_AMASS:AMASS_XT60-M_1x02_P7.20mm_Vertical -> Connector_AMASS:AMASS_XT30UPB-M_1x02_P5.0mm_Vertical
- J3: footprint Connector_AMASS:AMASS_XT60-F_1x02_P7.20mm_Vertical -> Connector_AMASS:AMASS_XT30UPB-M_1x02_P5.0mm_Vertical
- moved J2 3.88 mm to (154.9, 87.4)
- moved J3 2.84 mm to (163.9, 87.4)
Routing:
- net GND: track 17.2 -> 6.59 mm, vias 29 -> 37
Other:
- outline, holes or cut-outs redrawn
