File: NMOS_SWITCH.kicad_sch (KiCad schematic)
At the start: 22 parts, among them J1 Conn_01x02, J2 Conn_01x02, J3 Conn_01x02, Q1 Q_NPN_BCE, Q2 CSD18540Q5B, U1 BTS443P, U2 LM5050-1

Commit message: Adoption changes for engineering
Parts:
- added H2: MountingHole, MountingHole:MountingHole_3.2mm_M3, symbol Mechanical:MountingHole
- J2: footprint Connector_AMASS:AMASS_XT60-M_1x02_P7.20mm_Vertical -> Connector_AMASS:AMASS_XT30UPB-M_1x02_P5.0mm_Vertical
- J3: footprint Connector_AMASS:AMASS_XT60-F_1x02_P7.20mm_Vertical -> Connector_AMASS:AMASS_XT30UPB-M_1x02_P5.0mm_Vertical
Changed lines of the file:
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@@
     (property "Reference" "J2" (id 0) (at 52.07 31.75 0))
     (property "Value" "Conn_01x02" (id 1) (at 52.07 34.29 0))
-    (property "Footprint" "Connector_AMASS:AMASS_XT60-M_1x02_P7.20mm_Vertical" (id 2) (at 52.07 40.64 0)
+    (property "Footprint" "Connector_AMASS:AMASS_XT30UPB-M_1x02_P5.0mm_Vertical" (id 2) (at 52.07 40.64 0)
       (effects (font (size 1.27 1.27)) hide)
     )
@@
     )
     (pin "1")
+  )
+  (symbol (lib_id "Mechanical:MountingHole") (at 26.67 113.03 0) (unit 1)
+    (in_bom yes) (on_board yes) (fields_autoplaced)
+    (property "Reference" "H2" (id 0) (at 29.21 112.1215 0)
+      (effects (font (size 1.27 1.27)) (justify left))
+    )
+    (property "Value" "MountingHole" (id 1) (at 29.21 114.8966 0)
+      (effects (font (size 1.27 1.27)) (justify left))
+    )
+    (property "Footprint" "MountingHole:MountingHole_3.2mm_M3" (id 2) (at 26.67 113.03 0)
+      (effects (font (size 1.27 1.27)) hide)
+    )
+    (property "Datasheet" "~" (id 3) (at 26.67 113.03 0)
+      (effects (font (size 1.27 1.27)) hide)
+    )
   )
   (symbol (lib_id "power:GNDPWR") (at 81.28 43.18 0) (unit 1)
@@
     (property "Reference" "J3" (id 0) (at 73.66 31.75 0))
     (property "Value" "Conn_01x02" (id 1) (at 73.66 34.29 0))
-    (property "Footprint" "Connector_AMASS:AMASS_XT60-F_1x02_P7.20mm_Vertical" (id 2) (at 73.66 40.64 0)
+    (property "Footprint" "Connector_AMASS:AMASS_XT30UPB-M_1x02_P5.0mm_Vertical" (id 2) (at 73.66 40.64 0)
       (effects (font (size 1.27 1.27)) hide)
     )
@@
       (reference "H1") (unit 1) (value "MountingHole") (footprint "MountingHole:MountingHole_3.2mm_M3")
     )
+    (path "/42795956-f125-4166-860d-4316fe3791b8"
+      (reference "H2") (unit 1) (value "MountingHole") (footprint "MountingHole:MountingHole_3.2mm_M3")
+    )
     (path "/394d0d22-ad22-48a2-8a98-c70e90863c41"
       (reference "J1") (unit 1) (value "Conn_01x02") (footprint "Connector_AMASS:AMASS_XT30UPB-M_1x02_P5.0mm_Vertical")
     )
     (path "/3d81c21a-eaa8-415e-965e-1e947463fab8"
-      (reference "J2") (unit 1) (value "Conn_01x02") (footprint "Connector_AMASS:AMASS_XT60-M_1x02_P7.20mm_Vertical")
+      (reference "J2") (unit 1) (value "Conn_01x02") (footprint "Connector_AMASS:AMASS_XT30UPB-M_1x02_P5.0mm_Vertical")
     )
     (path "/b42b89a7-c059-4fa0-9ad0-405247d9a525"
-      (reference "J3") (unit 1) (value "Conn_01x02") (footprint "Connector_AMASS:AMASS_XT60-F_1x02_P7.20mm_Vertical")
+      (reference "J3") (unit 1) (value "Conn_01x02") (footprint "Connector_AMASS:AMASS_XT30UPB-M_1x02_P5.0mm_Vertical")
     )
     (path "/2b9f3e20-0ba7-4c69-ac3d-4d14e26945ec"

Commit message: Change some footprints
Parts:
- removed D4: SVM1550UB, POWER_DIODE_SMD:TO-277A, symbol Power_diode:SVM1550UB
Changed lines of the file:
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@@
 (kicad_sch (version 20211123) (generator eeschema)
   (paper "A4")
-  (junction (at 138.43 54.61) (diameter 0) (color 0 0 0 0)
-  )
   (junction (at 119.38 81.28) (diameter 0) (color 0 0 0 0)
   )
@@
     (stroke (width 0) (type default) (color 0 0 0 0))
   )
-  (wire (pts (xy 138.43 49.53) (xy 138.43 54.61))
-    (stroke (width 0) (type default) (color 0 0 0 0))
-  )
   (wire (pts (xy 77.47 66.04) (xy 77.47 62.23))
     (stroke (width 0) (type default) (color 0 0 0 0))
@@
     (stroke (width 0) (type default) (color 0 0 0 0))
   )
-  (wire (pts (xy 133.35 54.61) (xy 138.43 54.61))
-    (stroke (width 0) (type default) (color 0 0 0 0))
-  )
   (wire (pts (xy 151.13 64.77) (xy 162.56 64.77))
     (stroke (width 0) (type default) (color 0 0 0 0))
@@
     (stroke (width 0) (type default) (color 0 0 0 0))
   )
-  (wire (pts (xy 119.38 54.61) (xy 119.38 64.77))
-    (stroke (width 0) (type default) (color 0 0 0 0))
-  )
   (wire (pts (xy 160.02 83.82) (xy 162.56 83.82))
     (stroke (width 0) (type default) (color 0 0 0 0))
@@
     (stroke (width 0) (type default) (color 0 0 0 0))
   )
-  (wire (pts (xy 119.38 54.61) (xy 123.19 54.61))
-    (stroke (width 0) (type default) (color 0 0 0 0))
-  )
   (wire (pts (xy 109.22 88.9) (xy 109.22 92.71))
     (stroke (width 0) (type default) (color 0 0 0 0))
   )
-  (wire (pts (xy 138.43 54.61) (xy 138.43 64.77))
+  (wire (pts (xy 138.43 49.53) (xy 138.43 64.77))
     (stroke (width 0) (type default) (color 0 0 0 0))
   )
@@
     )
     (pin "1")
-  )
-  (symbol (lib_id "Power_diode:SVM1550UB") (at 128.27 54.61 180) (unit 1)
-    (in_bom yes) (on_board yes) (fields_autoplaced)
-    (property "Reference" "D4" (id 0) (at 128.27 48.26 0))
-    (property "Value" "SVM1550UB" (id 1) (at 128.27 50.8 0))
-    (property "Footprint" "POWER_DIODE_SMD:TO-277A" (id 2) (at 107.95 57.15 0)
-      (effects (font (size 1.27 1.27)) hide)
-    )
-    (property "Datasheet" "" (id 3) (at 128.27 54.61 0)
-      (effects (font (size 1.27 1.27)) hide)
-    )
-    (pin "A")
-    (pin "K")
   )
   (symbol (lib_id "Basic_passive_components:Resistor") (at 101.6 76.2 0) (unit 1)
@@
       (reference "D3") (unit 1) (value "LED") (footprint "LED_SMD:LED_0603_1608Metric")
     )
-    (path "/74420387-a722-44a9-bcc2-30f2d49e18a4"
-      (reference "D4") (unit 1) (value "SVM1550UB") (footprint "POWER_DIODE_SMD:TO-277A")
-    )
     (path "/afdca86f-c245-4e1f-a619-e486c086bb0e"
